Commit message: Values im currently using in my experiments

File: yumi_description/urdf/Extras/yumi_optodaq_sensors.xacro (robot description, xacro)
@@ -3,5 +3,5 @@
   <xacro:macro name="yumi_optodaq_sensor" params="parent name *origin">
     <!--joint between {parent} and base-->
-    <joint name="${parent}_joint" type="fixed">
+    <joint name="${parent}_joint_daq" type="fixed">
       <xacro:insert_block name="origin"/>
       <parent link="${parent}"/>

File: yumi_description/urdf/yumi.urdf (robot description, URDF)
Before this commit: robot yumi, 24 links, 23 joints
Links:
- link gripper_l_finger_l: mass 0.01 -> 0.1
- link gripper_l_finger_r: mass 0.01 -> 0.1
- link gripper_r_finger_l: mass 0.01 -> 0.1
- link gripper_r_finger_r: mass 0.01 -> 0.1
