Commit message: Integrated optoforce sensors in YuMi URDF

File: yumi_description/urdf/yumi.urdf.xacro (robot description, xacro)
@@ -17,22 +17,16 @@
     <origin xyz="0 0 0.1" rpy="0 0 0" />
   </xacro:yumi>
-  <!--right gripper-->
-  <xacro:yumi_servo_gripper name="gripper_r" hardware_interface="hardware_interface/$(arg grippers_interface)" parent="${gripper_r_parent}">
-    <origin xyz="0 0 ${gripper_base_z}" rpy="0 0 ${PI}" />
-  </xacro:yumi_servo_gripper>
-  <!--left gripper-->
-  <xacro:yumi_servo_gripper name="gripper_l" hardware_interface="hardware_interface/$(arg grippers_interface)" parent="${gripper_l_parent}">
-    <origin xyz="0 0 ${gripper_base_z}" rpy="0 0 ${PI}" />
-  </xacro:yumi_servo_gripper>
-  <xacro:property name="optodaq" value="$(arg optodaq_sensors)" />
-  <xacro:if value="${optodaq == 'false'}">
-	<xacro:property name="gripper_r_parent" value="yumi_link_7_r" />
-	<xacro:property name="gripper_l_parent" value="yumi_link_7_l" />
-	<xacro:property name="gripper_base_z" value="0.007" />
+  <xacro:property name="optodaq_sensors" value="$(arg optodaq_sensors)" />
+  <xacro:if value="${optodaq_sensors == 'false'}">
+	<!--right gripper-->
+	<xacro:yumi_servo_gripper name="gripper_r" hardware_interface="hardware_interface/$(arg grippers_interface)" parent="yumi_link_7_r">
+		<origin xyz="0 0 0.007" rpy="0 0 ${PI}" />
+	</xacro:yumi_servo_gripper>
+	<!--left gripper-->
+	<xacro:yumi_servo_gripper name="gripper_l" hardware_interface="hardware_interface/$(arg grippers_interface)" parent="yumi_link_7_l">
+		<origin xyz="0 0 0.007" rpy="0 0 ${PI}" />
+	</xacro:yumi_servo_gripper>
   </xacro:if>
-<!--   <xacro:if value="${optodaq == 'true'}">
-	  <xacro:property name="gripper_r_parent" value="optodaq_r_sensor_link" />
-	  <xacro:property name="gripper_l_parent" value="optodaq_l_sensor_link" />
-	  <xacro:property name="gripper_base_z" value="0.033" />
+  <xacro:if value="${optodaq_sensors == 'true'}">
 	  <xacro:yumi_optodaq_sensor name="optodaq_r" parent="yumi_link_7_r">
 	    <origin xyz="0 0 0.033" rpy="0 0 ${PI}" />
@@ -41,6 +35,13 @@
 	    <origin xyz="0 0 0.033" rpy="0 0 ${PI}" />
 	  </xacro:yumi_optodaq_sensor>
+	<!--right gripper-->
+	<xacro:yumi_servo_gripper name="gripper_r" hardware_interface="hardware_interface/$(arg grippers_interface)" parent="optodaq_r_sensor_link">
+		<origin xyz="0 0 0.033" rpy="0 0 ${PI}" />
+	</xacro:yumi_servo_gripper>
+	<!--left gripper-->
+	<xacro:yumi_servo_gripper name="gripper_l" hardware_interface="hardware_interface/$(arg grippers_interface)" parent="optodaq_l_sensor_link">
+		<origin xyz="0 0 0.033" rpy="0 0 ${PI}" />
+	</xacro:yumi_servo_gripper>
   </xacro:if>
- -->
   <xacro:property name="yumi_setup" value="$(arg yumi_setup)" />
   <xacro:if value="${yumi_setup == 'robot_centric'}">

Commit message: Updating the YuMi launch files to integrate the Optoforce 6 axis sensors

File: yumi_description/urdf/yumi.urdf.xacro (robot description, xacro)
@@ -29,18 +29,18 @@
   </xacro:if>
   <xacro:if value="${optodaq_sensors == 'true'}">
-	  <xacro:yumi_optodaq_sensor name="optodaq_r" parent="yumi_link_7_r">
-	    <origin xyz="0 0 0.033" rpy="0 0 ${PI}" />
-	  </xacro:yumi_optodaq_sensor>
-	  <xacro:yumi_optodaq_sensor name="optodaq_l" parent="yumi_link_7_l">
-	    <origin xyz="0 0 0.033" rpy="0 0 ${PI}" />
-	  </xacro:yumi_optodaq_sensor>
-	<!--right gripper-->
-	<xacro:yumi_servo_gripper name="gripper_r" hardware_interface="hardware_interface/$(arg grippers_interface)" parent="optodaq_r_sensor_link">
-		<origin xyz="0 0 0.033" rpy="0 0 ${PI}" />
-	</xacro:yumi_servo_gripper>
-	<!--left gripper-->
-	<xacro:yumi_servo_gripper name="gripper_l" hardware_interface="hardware_interface/$(arg grippers_interface)" parent="optodaq_l_sensor_link">
-		<origin xyz="0 0 0.033" rpy="0 0 ${PI}" />
-	</xacro:yumi_servo_gripper>
+    <xacro:yumi_optodaq_sensor name="optodaq_r" parent="yumi_link_7_r">
+      <origin xyz="0 0 0.033" rpy="0 0 ${PI}" />
+    </xacro:yumi_optodaq_sensor>
+    <xacro:yumi_optodaq_sensor name="optodaq_l" parent="yumi_link_7_l">
+      <origin xyz="0 0 0.033" rpy="0 0 ${PI}" />
+    </xacro:yumi_optodaq_sensor>
+    <!--right gripper-->
+    <xacro:yumi_servo_gripper name="gripper_r" hardware_interface="hardware_interface/$(arg grippers_interface)" parent="optodaq_r_sensor_link">
+      <origin xyz="0 0 0.033" rpy="0 0 ${PI}" />
+    </xacro:yumi_servo_gripper>
+    <!--left gripper-->
+    <xacro:yumi_servo_gripper name="gripper_l" hardware_interface="hardware_interface/$(arg grippers_interface)" parent="optodaq_l_sensor_link">
+      <origin xyz="0 0 0.033" rpy="0 0 ${PI}" />
+    </xacro:yumi_servo_gripper>
   </xacro:if>
   <xacro:property name="yumi_setup" value="$(arg yumi_setup)" />

Commit message: Reverting Optoforce sensors integration changes. From now on they will be done in a different branch

File: yumi_description/urdf/yumi.urdf.xacro (robot description, xacro)
@@ -9,6 +9,4 @@
   <!--Import the yumi servo gripper macro -->
   <xacro:include filename="$(find yumi_description)/urdf/Grippers/yumi_servo_gripper.xacro"/>
-  <!--Import the yumi optodaq sensors macro -->
-  <xacro:include filename="$(find yumi_description)/urdf/Extras/yumi_optodaq_sensors.xacro"/>
   <!-- Import Gazebo plugins -->
   <xacro:include filename="$(find yumi_description)/urdf/Gazebo/gazebo.urdf.xacro"/>
@@ -18,29 +16,11 @@
   </xacro:yumi>
   <!--right gripper-->
-  <xacro:yumi_servo_gripper name="gripper_r" hardware_interface="hardware_interface/$(arg grippers_interface)" parent="${gripper_r_parent}">
-    <origin xyz="0 0 ${gripper_base_z}" rpy="0 0 ${PI}" />
+  <xacro:yumi_servo_gripper name="gripper_r" hardware_interface="hardware_interface/$(arg grippers_interface)" parent="yumi_link_7_r">
+    <origin xyz="0 0 0.007" rpy="0 0 ${PI}" />
   </xacro:yumi_servo_gripper>
   <!--left gripper-->
-  <xacro:yumi_servo_gripper name="gripper_l" hardware_interface="hardware_interface/$(arg grippers_interface)" parent="${gripper_l_parent}">
-    <origin xyz="0 0 ${gripper_base_z}" rpy="0 0 ${PI}" />
+  <xacro:yumi_servo_gripper name="gripper_l" hardware_interface="hardware_interface/$(arg grippers_interface)" parent="yumi_link_7_l">
+    <origin xyz="0 0 0.007" rpy="0 0 ${PI}" />
   </xacro:yumi_servo_gripper>
-  <xacro:property name="optodaq" value="$(arg optodaq_sensors)" />
-  <xacro:if value="${optodaq == 'false'}">
-	<xacro:property name="gripper_r_parent" value="yumi_link_7_r" />
-	<xacro:property name="gripper_l_parent" value="yumi_link_7_l" />
-	<xacro:property name="gripper_base_z" value="0.007" />
-  </xacro:if>
-<!--   <xacro:if value="${optodaq == 'true'}">
-	  <xacro:property name="gripper_r_parent" value="optodaq_r_sensor_link" />
-	  <xacro:property name="gripper_l_parent" value="optodaq_l_sensor_link" />
-	  <xacro:property name="gripper_base_z" value="0.033" />
-	  <xacro:yumi_optodaq_sensor name="optodaq_r" parent="yumi_link_7_r">
-	    <origin xyz="0 0 0.033" rpy="0 0 ${PI}" />
-	  </xacro:yumi_optodaq_sensor>
-	  <xacro:yumi_optodaq_sensor name="optodaq_l" parent="yumi_link_7_l">
-	    <origin xyz="0 0 0.033" rpy="0 0 ${PI}" />
-	  </xacro:yumi_optodaq_sensor>
-  </xacro:if>
- -->
   <xacro:property name="yumi_setup" value="$(arg yumi_setup)" />
   <xacro:if value="${yumi_setup == 'robot_centric'}">

Commit message: fixed gripper orientation in the urdf

File: yumi_description/urdf/yumi.urdf.xacro (robot description, xacro)
@@ -18,16 +18,16 @@
   </xacro:yumi>
   <xacro:yumi_optodaq_sensor name="optodaq_r" parent="yumi_link_7_r">
-    <origin xyz="0 0 0.033" rpy="0 0 ${PI}" />
+    <origin xyz="0 0 0.033" rpy="0 ${PI} -0.7" />
   </xacro:yumi_optodaq_sensor>
   <xacro:yumi_optodaq_sensor name="optodaq_l" parent="yumi_link_7_l">
-    <origin xyz="0 0 0.033" rpy="0 0 ${PI}" />
+    <origin xyz="0 0 0.033" rpy="0 ${PI} -0.7" />
   </xacro:yumi_optodaq_sensor>
   <!--right gripper-->
-  <xacro:yumi_servo_gripper name="gripper_r" hardware_interface="hardware_interface/$(arg grippers_interface)" parent="optodaq_r_sensor_link">
-    <origin xyz="0 0 0.033" rpy="0 0 ${PI}" />
+  <xacro:yumi_servo_gripper name="gripper_r" hardware_interface="hardware_interface/EffortJointInterface" parent="optodaq_r_sensor_link">
+    <origin xyz="0 0 -0.033" rpy="${PI} 0.0 ${PI/4}" />
   </xacro:yumi_servo_gripper>
   <!--left gripper-->
-  <xacro:yumi_servo_gripper name="gripper_l" hardware_interface="hardware_interface/$(arg grippers_interface)" parent="optodaq_l_sensor_link">
-    <origin xyz="0 0 0.033" rpy="0 0 ${PI}" />
+  <xacro:yumi_servo_gripper name="gripper_l" hardware_interface="hardware_interface/EffortJointInterface" parent="optodaq_l_sensor_link">
+    <origin xyz="0 0 -0.033" rpy="${PI} 0.0 ${PI/4}" />
   </xacro:yumi_servo_gripper>
   <xacro:property name="yumi_setup" value="$(arg yumi_setup)" />

Commit message: urdf update

File: yumi_description/urdf/yumi.urdf.xacro (robot description, xacro)
@@ -18,8 +18,8 @@
   </xacro:yumi>
   <xacro:yumi_optodaq_sensor name="optodaq_r" parent="yumi_link_7_r">
-    <origin xyz="0 0 0.033" rpy="0 ${PI} -0.7" />
+    <origin xyz="0 0 0.033" rpy="0 ${PI} ${-PI/4}" />
   </xacro:yumi_optodaq_sensor>
   <xacro:yumi_optodaq_sensor name="optodaq_l" parent="yumi_link_7_l">
-    <origin xyz="0 0 0.033" rpy="0 ${PI} -0.7" />
+    <origin xyz="0 0 0.033" rpy="0 ${PI} ${-PI/4}" />
   </xacro:yumi_optodaq_sensor>
   <!--right gripper-->

Commit message: urdf tweak

File: yumi_description/urdf/yumi.urdf.xacro (robot description, xacro)
@@ -17,18 +17,18 @@
     <origin xyz="0 0 0.1" rpy="0 0 0" />
   </xacro:yumi>
-  <xacro:yumi_optodaq_sensor name="optodaq_r" parent="yumi_link_7_r">
-    <origin xyz="0 0 0.033" rpy="0 ${PI} ${-PI/4}" />
-  </xacro:yumi_optodaq_sensor>
-  <xacro:yumi_optodaq_sensor name="optodaq_l" parent="yumi_link_7_l">
-    <origin xyz="0 0 0.033" rpy="0 ${PI} ${-PI/4}" />
-  </xacro:yumi_optodaq_sensor>
-  <!--right gripper-->
-  <xacro:yumi_servo_gripper name="gripper_r" hardware_interface="hardware_interface/EffortJointInterface" parent="optodaq_r_sensor_link">
-    <origin xyz="0 0 -0.033" rpy="${PI} 0.0 ${PI/4}" />
-  </xacro:yumi_servo_gripper>
-  <!--left gripper-->
-  <xacro:yumi_servo_gripper name="gripper_l" hardware_interface="hardware_interface/EffortJointInterface" parent="optodaq_l_sensor_link">
-    <origin xyz="0 0 -0.033" rpy="${PI} 0.0 ${PI/4}" />
-  </xacro:yumi_servo_gripper>
+ <xacro:yumi_optodaq_sensor name="optodaq_r" parent="yumi_link_7_r">
+     <origin xyz="0 0 0.033" rpy="0 ${PI} ${-PI/4}" />
+ </xacro:yumi_optodaq_sensor>
+ <xacro:yumi_optodaq_sensor name="optodaq_l" parent="yumi_link_7_l">
+   <origin xyz="0 0 0.033" rpy="0 ${PI} ${-PI/4}" />
+ </xacro:yumi_optodaq_sensor>
+ <!--right gripper-->
+ <xacro:yumi_servo_gripper name="gripper_r" hardware_interface="hardware_interface/EffortJointInterface" parent="optodaq_r_sensor_link">
+   <origin xyz="0 0 -0.033" rpy="${PI} 0.0 ${PI/4}" />
+ </xacro:yumi_servo_gripper>
+ <!--left gripper-->
+ <xacro:yumi_servo_gripper name="gripper_l" hardware_interface="hardware_interface/EffortJointInterface" parent="optodaq_l_sensor_link">
+   <origin xyz="0 0 -0.033" rpy="${PI} 0.0 ${PI/4}" />
+ </xacro:yumi_servo_gripper>
   <xacro:property name="yumi_setup" value="$(arg yumi_setup)" />
   <xacro:if value="${yumi_setup == 'robot_centric'}">

Commit message: Taking out meshes and code from the URDF that should be only in the specific project branches

File: yumi_description/urdf/yumi.urdf.xacro (robot description, xacro)
@@ -36,137 +36,3 @@
     </joint>
   </xacro:if>
-  <xacro:if value="${yumi_setup == 'AUTOMED'}">
-    <xacro:property name="pedestal_height" value="0.92" />
-    <xacro:property name="pedestal_xrotation_fix" value="${- PI / 2.0}" />
-    <xacro:property name="pedestal_zrotation_fix" value="${PI}" />
-    <xacro:property name="yumi_offset_x" value="-0.0625" />
-    <xacro:property name="yumi_height" value="0.04" />
-    <xacro:property name="yumi_parent" value="yumi_pedestal" />
-    <link name="world"/>
-    <joint name="world_to_pedestal" type="fixed">
-      <parent link="world" />
-      <child link="yumi_pedestal" />
-      <origin rpy="0 0 0" xyz="0 0 ${pedestal_height}" />
-    </joint>
-    <link name="yumi_pedestal">
-<!--       <collision>
-        <origin xyz="0 0 0" rpy="${pedestal_xrotation_fix} 0 ${pedestal_zrotation_fix}" />
-        <geometry>
-          <mesh scale="0.001 0.001 0.001" filename="package://yumi_description/meshes/accesories/KTH_AutoMed_Aluflex_pedestal.stl"/>
-        </geometry>
-        <material name="Grey" />
-      </collision> -->
-      <visual>
-        <origin xyz="0 0 0" rpy="${pedestal_xrotation_fix} 0 ${pedestal_zrotation_fix}" />
-        <geometry>
-          <mesh scale="0.001 0.001 0.001" filename="package://yumi_description/meshes/accesories/KTH_AutoMed_Aluflex_pedestal.stl"/>
-        </geometry>
-        <material name="Grey" />
-      </visual>
-    </link>
-    <joint name="pedestal_to_yumi" type="fixed">
-      <parent link="yumi_pedestal" />
-      <child link="yumi_base_link" />
-      <origin rpy="0 0 0" xyz="${yumi_offset_x} 0 ${yumi_height}" />
-    </joint>
-  </xacro:if>
-  <xacro:if value="${yumi_setup == 'FACT'}">
-    <xacro:property name="pedestal_height" value="0.92" />
-    <xacro:property name="pedestal_xrotation_fix" value="${- PI / 2.0}" />
-    <xacro:property name="pedestal_zrotation_fix" value="${PI}" />
-    <xacro:property name="yumi_offset_x" value="-0.0625" />
-    <xacro:property name="yumi_height" value="0.04" />
-    <xacro:property name="yumi_parent" value="yumi_pedestal" />
-    <xacro:property name="kinect_zrotation_fix" value="${- PI / 2.0}" />
-    <link name="world"/>
-    <joint name="world_to_pedestal" type="fixed">
-      <parent link="world" />
-      <child link="yumi_pedestal" />
-      <origin rpy="0 0 0" xyz="0 0 ${pedestal_height}" />
-    </joint>
-    <link name="yumi_pedestal">
-      <visual>
-        <origin xyz="0 0 0" rpy="${pedestal_xrotation_fix} 0 ${pedestal_zrotation_fix}" />
-        <geometry>
-          <mesh scale="0.001 0.001 0.001" filename="package://yumi_description/meshes/accesories/KTH_AutoMed_Aluflex_pedestal.stl"/>
-        </geometry>
-        <material name="Grey" />
-      </visual>
-    </link>
-    <joint name="pedestal_to_table" type="fixed">
-      <parent link="yumi_pedestal" />
-      <child link="table" />
-      <origin rpy="0 0 0" xyz="0.235 0 ${yumi_height}" />
-    </joint>
-    <link name="table">
-        <visual>
-          <origin xyz="0 0 0" rpy="0 0 0" />
-          <geometry>
-            <box size="0.6 0.6 0.02" />
-          </geometry>
-          <material name="Grey" />
-        </visual>
-    </link>
-    <joint name="pedestal_to_yumi" type="fixed">
-      <parent link="yumi_pedestal" />
-      <child link="yumi_base_link" />
-      <origin rpy="0 0 0" xyz="${yumi_offset_x} 0 ${yumi_height+0.02}" />
-    </joint>
-    <link name="kinect2">
-      <visual>
-        <origin xyz="0 0 0" rpy="0 0 0" />
-        <geometry>
-          <mesh scale="0.001 0.001 0.001" filename="package://yumi_description/meshes/accesories/KinectXboxOne.stl"/>
-        </geometry>
-        <material name="Black" />
-      </visual>
-    </link>
-    <link name="left_kinect_base">
-        <visual>
-          <origin xyz="0 0 0" rpy="0 0 0" />
-          <geometry>
-            <box size="0.4 0.02 0.02" />
-          </geometry>
-          <material name="Grey" />
-        </visual>
-    </link>
-    <link name="right_kinect_base">
-        <visual>
-          <origin xyz="0 0 0" rpy="0 0 0" />
-          <geometry>
-            <box size="0.4 0.02 0.02" />
-          </geometry>
-          <material name="Grey" />
-        </visual>
-    </link>
-    <link name="middle_kinect_base">
-        <visual>
-          <origin xyz="0 0 0" rpy="0 0 0" />
-          <geometry>
-            <box size="0.4 0.02 0.02" />
-          </geometry>
-          <material name="Grey" />
-        </visual>
-    </link>
-     <joint name="kinect2_to_right_kinect_base" type="fixed">
-      <parent link="yumi_base_link" />
-      <child link="right_kinect_base" />
-      <origin rpy="0 ${-PI/6} 0.17" xyz="0.1 -0.03 0.56" />
-    </joint>
-    <joint name="kinect2_to_left_kinect_base" type="fixed">
-      <parent link="yumi_base_link" />
-      <child link="left_kinect_base" />
-      <origin rpy="0 ${-PI/6} -0.17" xyz="0.1 0.03 0.56" />
-    </joint>
-    <joint name="yumi_to_middle_kinect_base" type="fixed">
-      <parent link="yumi_base_link" />
-      <child link="middle_kinect_base" />
-      <origin rpy="0 ${-PI/6} 0" xyz="0.05 0 0.56" />
-    </joint>
-    <joint name="middle_kinect_base_to_kinect2" type="fixed">
-      <parent link="middle_kinect_base" />
-      <child link="kinect2" />
-      <origin rpy="${-PI/2} 0 ${kinect_zrotation_fix}" xyz="0.2 0 0" />
-    </joint>
-  </xacro:if>
 </robot>

Commit message: DIrect integration of Optoforce 6axis F/T sensors into YuMi hardware interface

File: yumi_description/urdf/yumi.urdf.xacro (robot description, xacro)
@@ -44,137 +44,3 @@
     </joint>
   </xacro:if>
-  <xacro:if value="${yumi_setup == 'AUTOMED'}">
-    <xacro:property name="pedestal_height" value="0.92" />
-    <xacro:property name="pedestal_xrotation_fix" value="${- PI / 2.0}" />
-    <xacro:property name="pedestal_zrotation_fix" value="${PI}" />
-    <xacro:property name="yumi_offset_x" value="-0.0625" />
-    <xacro:property name="yumi_height" value="0.04" />
-    <xacro:property name="yumi_parent" value="yumi_pedestal" />
-    <link name="world"/>
-    <joint name="world_to_pedestal" type="fixed">
-      <parent link="world" />
-      <child link="yumi_pedestal" />
-      <origin rpy="0 0 0" xyz="0 0 ${pedestal_height}" />
-    </joint>
-    <link name="yumi_pedestal">
-<!--       <collision>
-        <origin xyz="0 0 0" rpy="${pedestal_xrotation_fix} 0 ${pedestal_zrotation_fix}" />
-        <geometry>
-          <mesh scale="0.001 0.001 0.001" filename="package://yumi_description/meshes/accesories/KTH_AutoMed_Aluflex_pedestal.stl"/>
-        </geometry>
-        <material name="Grey" />
-      </collision> -->
-      <visual>
-        <origin xyz="0 0 0" rpy="${pedestal_xrotation_fix} 0 ${pedestal_zrotation_fix}" />
-        <geometry>
-          <mesh scale="0.001 0.001 0.001" filename="package://yumi_description/meshes/accesories/KTH_AutoMed_Aluflex_pedestal.stl"/>
-        </geometry>
-        <material name="Grey" />
-      </visual>
-    </link>
-    <joint name="pedestal_to_yumi" type="fixed">
-      <parent link="yumi_pedestal" />
-      <child link="yumi_base_link" />
-      <origin rpy="0 0 0" xyz="${yumi_offset_x} 0 ${yumi_height}" />
-    </joint>
-  </xacro:if>
-  <xacro:if value="${yumi_setup == 'FACT'}">
-    <xacro:property name="pedestal_height" value="0.92" />
-    <xacro:property name="pedestal_xrotation_fix" value="${- PI / 2.0}" />
-    <xacro:property name="pedestal_zrotation_fix" value="${PI}" />
-    <xacro:property name="yumi_offset_x" value="-0.0625" />
-    <xacro:property name="yumi_height" value="0.04" />
-    <xacro:property name="yumi_parent" value="yumi_pedestal" />
-    <xacro:property name="kinect_zrotation_fix" value="${- PI / 2.0}" />
-    <link name="world"/>
-    <joint name="world_to_pedestal" type="fixed">
-      <parent link="world" />
-      <child link="yumi_pedestal" />
-      <origin rpy="0 0 0" xyz="0 0 ${pedestal_height}" />
-    </joint>
-    <link name="yumi_pedestal">
-      <visual>
-        <origin xyz="0 0 0" rpy="${pedestal_xrotation_fix} 0 ${pedestal_zrotation_fix}" />
-        <geometry>
-          <mesh scale="0.001 0.001 0.001" filename="package://yumi_description/meshes/accesories/KTH_AutoMed_Aluflex_pedestal.stl"/>
-        </geometry>
-        <material name="Grey" />
-      </visual>
-    </link>
-    <joint name="pedestal_to_table" type="fixed">
-      <parent link="yumi_pedestal" />
-      <child link="table" />
-      <origin rpy="0 0 0" xyz="0.235 0 ${yumi_height}" />
-    </joint>
-    <link name="table">
-        <visual>
-          <origin xyz="0 0 0" rpy="0 0 0" />
-          <geometry>
-            <box size="0.6 0.6 0.02" />
-          </geometry>
-          <material name="Grey" />
-        </visual>
-    </link>
-    <joint name="pedestal_to_yumi" type="fixed">
-      <parent link="yumi_pedestal" />
-      <child link="yumi_base_link" />
-      <origin rpy="0 0 0" xyz="${yumi_offset_x} 0 ${yumi_height+0.02}" />
-    </joint>
-    <link name="kinect2">
-      <visual>
-        <origin xyz="0 0 0" rpy="0 0 0" />
-        <geometry>
-          <mesh scale="0.001 0.001 0.001" filename="package://yumi_description/meshes/accesories/KinectXboxOne.stl"/>
-        </geometry>
-        <material name="Black" />
-      </visual>
-    </link>
-    <link name="left_kinect_base">
-        <visual>
-          <origin xyz="0 0 0" rpy="0 0 0" />
-          <geometry>
-            <box size="0.4 0.02 0.02" />
-          </geometry>
-          <material name="Grey" />
-        </visual>
-    </link>
-    <link name="right_kinect_base">
-        <visual>
-          <origin xyz="0 0 0" rpy="0 0 0" />
-          <geometry>
-            <box size="0.4 0.02 0.02" />
-          </geometry>
-          <material name="Grey" />
-        </visual>
-    </link>
-    <link name="middle_kinect_base">
-        <visual>
-          <origin xyz="0 0 0" rpy="0 0 0" />
-          <geometry>
-            <box size="0.4 0.02 0.02" />
-          </geometry>
-          <material name="Grey" />
-        </visual>
-    </link>
-     <joint name="kinect2_to_right_kinect_base" type="fixed">
-      <parent link="yumi_base_link" />
-      <child link="right_kinect_base" />
-      <origin rpy="0 ${-PI/6} 0.17" xyz="0.1 -0.03 0.56" />
-    </joint>
-    <joint name="kinect2_to_left_kinect_base" type="fixed">
-      <parent link="yumi_base_link" />
-      <child link="left_kinect_base" />
-      <origin rpy="0 ${-PI/6} -0.17" xyz="0.1 0.03 0.56" />
-    </joint>
-    <joint name="yumi_to_middle_kinect_base" type="fixed">
-      <parent link="yumi_base_link" />
-      <child link="middle_kinect_base" />
-      <origin rpy="0 ${-PI/6} 0" xyz="0.05 0 0.56" />
-    </joint>
-    <joint name="middle_kinect_base_to_kinect2" type="fixed">
-      <parent link="middle_kinect_base" />
-      <child link="kinect2" />
-      <origin rpy="${-PI/2} 0 ${kinect_zrotation_fix}" xyz="0.2 0 0" />
-    </joint>
-  </xacro:if>
 </robot>
