Commit message: fixed yumi gripper_r orientation for the new mount

File: yumi_description/urdf/yumi.urdf.xacro (robot description, xacro)
@@ -18,5 +18,5 @@
   </xacro:yumi>
  <xacro:yumi_optodaq_sensor name="optodaq_r" parent="yumi_link_7_r">
-     <origin xyz="0 0 0.033" rpy="0 ${PI} ${-PI/4}" />
+   <origin xyz="0 0 0.033" rpy="0 0 ${5*PI/8}" />
  </xacro:yumi_optodaq_sensor>
  <xacro:yumi_optodaq_sensor name="optodaq_l" parent="yumi_link_7_l">
@@ -25,5 +25,5 @@
  <!--right gripper-->
  <xacro:yumi_servo_gripper name="gripper_r" hardware_interface="hardware_interface/EffortJointInterface" parent="optodaq_r_sensor_link">
-   <origin xyz="0 0 -0.033" rpy="${PI} 0.0 ${PI/4}" />
+   <origin xyz="0 0 0.033" rpy="${PI} 0.0 ${PI/4}" />
  </xacro:yumi_servo_gripper>
  <!--left gripper-->

Commit message: Being able to control the robot through RWS. Modified the makefile to have gazebo_mimic compiled. Also modified yumi.urdf.xarco, launch files, and files (*.h and *.cpp) under yumi_hw

File: yumi_description/urdf/yumi.urdf.xacro (robot description, xacro)
@@ -12,4 +12,5 @@
   <xacro:include filename="$(find yumi_description)/urdf/Gazebo/gazebo.urdf.xacro"/>
   <!--yumi-->
+  <xacro:property name="yumi_parent" value="world" />
   <xacro:yumi name="yumi" hardware_interface="hardware_interface/$(arg arms_interface)" parent="${yumi_parent}" >
     <origin xyz="0 0 0.1" rpy="0 0 0" />
