Commit message: Updated MoveIt! config for the new setup

File: yumi_description/urdf/yumi.urdf (robot description, URDF)
Before this commit: robot yumi, 28 links, 27 joints
Links:
- removed link left_kinect_base
- removed link right_kinect_base
- added link table_extension_bottom; visual mesh filename=package://yumi_description/meshes/accesories/tableExtension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 scale=0.001 0.001 0.001
- added link table_extension_top; visual mesh filename=package://yumi_description/meshes/accesories/tableExtension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 scale=0.001 0.001 0.001
- link middle_kinect_base: geometry visual box size=0.4 0.15 0.02
- link table: geometry visual mesh filename=package://yumi_description/meshes/accesories/steelTable.stl scale=0.001 0.001 0.001
Joints:
- removed joint kinect2_to_left_kinect_base
- removed joint kinect2_to_right_kinect_base
- added joint table_extension_bottom_to_top: type fixed, parent table_extension_bottom, child table_extension_top, origin xyz=0 0 0.005 rpy=0 0 0
- added joint table_to_extension_bottom: type fixed, parent table, child table_extension_bottom, origin xyz=0.75 -0.71 0.001 rpy=0 0 0
- joint pedestal_to_table: origin xyz=0.235 0 0.04 rpy=0 0 0 -> xyz=-0.05 0.235 0.05 rpy=0 0 0
- joint pedestal_to_yumi: origin xyz=-0.0625 0 0.06 rpy=0 0 0 -> xyz=-0.0625 0 0.05 rpy=0 0 0
- joint yumi_to_middle_kinect_base: origin xyz=0.05 0 0.56 rpy=0 -0.523598775598 0 -> xyz=-0.03 0 0.56 rpy=0 -1.25663706144 0

File: yumi_description/urdf/yumi.urdf.xacro (robot description, xacro)
@@ -63,5 +63,5 @@
 	      <material name="Grey" />
 	    </visual>
-	    <collision>
+<!-- 	    <collision>
 	      <origin xyz="0 0 0" rpy="${-PI/2} 0 ${-PI/2}" />
 	      <geometry>
@@ -69,5 +69,5 @@
 	      </geometry>
 	      <material name="Grey" />
-	    </collision>
+	    </collision> -->
 	</link>
 	<joint name="table_to_extension_bottom" type="fixed">
@@ -84,5 +84,5 @@
 	      <material name="Grey" />
 	    </visual>
-	    <collision>
+<!-- 	    <collision>
 	      <origin xyz="0 0 0" rpy="0 0 ${PI/2}" />
 	      <geometry>
@@ -90,5 +90,5 @@
 	      </geometry>
 	      <material name="Grey" />
-	    </collision>
+	    </collision> -->
 	</link>
 	<joint name="table_extension_bottom_to_top" type="fixed">
@@ -105,5 +105,5 @@
 	      <material name="White" />
 	    </visual>
-	    <collision>
+<!-- 	    <collision>
 	      <origin xyz="0 0 0" rpy="0 0 ${PI/2}" />
 	      <geometry>
@@ -111,5 +111,5 @@
 	      </geometry>
 	      <material name="White" />
-	    </collision>
+	    </collision> -->
 	</link>
 	<joint name="pedestal_to_yumi" type="fixed">
@@ -126,5 +126,5 @@
 	    <material name="Black" />
 	  </visual>
-	  <collision>
+<!-- 	  <collision>
 	    <origin xyz="0 0 0" rpy="0 0 0" />
 	    <geometry>
@@ -132,37 +132,5 @@
 	    </geometry>
 	    <material name="Black" />
-	  </collision>
-	</link>
-	<link name="left_kinect_base">
-	    <visual>
-	      <origin xyz="0 0 0" rpy="0 0 0" />
-	      <geometry>
-	        <box size="0.2 0.02 0.02" />
-	      </geometry>
-	      <material name="Grey" />
-	    </visual>
-	    <collision>
-	      <origin xyz="0 0 0" rpy="0 0 0" />
-	      <geometry>
-	        <box size="0.2 0.02 0.02" />
-	      </geometry>
-	      <material name="Grey" />
-	    </collision>
-	</link>
-	<link name="right_kinect_base">
-	    <visual>
-	      <origin xyz="0 0 0" rpy="0 0 0" />
-	      <geometry>
-	        <box size="0.2 0.02 0.02" />
-	      </geometry>
-	      <material name="Grey" />
-	    </visual>
-	    <collision>
-	      <origin xyz="0 0 0" rpy="0 0 0" />
-	      <geometry>
-	        <box size="0.2 0.02 0.02" />
-	      </geometry>
-	      <material name="Grey" />
-	    </collision>
+	  </collision> -->
 	</link>
 	<link name="middle_kinect_base">
@@ -170,30 +138,20 @@
 	      <origin xyz="0 0 0" rpy="0 0 0" />
 	      <geometry>
-	        <box size="0.4 0.02 0.02" />
+	        <box size="0.4 0.15 0.02" />
 	      </geometry>
 	      <material name="Grey" />
 	    </visual>
-	    <collision>
+<!-- 	    <collision>
 	      <origin xyz="0 0 0" rpy="0 0 0" />
 	      <geometry>
-	        <box size="0.4 0.02 0.02" />
+	        <box size="0.4 0.15 0.02" />
 	      </geometry>
 	      <material name="Grey" />
-	    </collision>
+	    </collision> -->
 	</link>
-	 <joint name="kinect2_to_right_kinect_base" type="fixed">
-	  <parent link="middle_kinect_base" />
-	  <child link="right_kinect_base" />
-	  <origin rpy="${PI/2} ${0.8*PI/2} 0" xyz="0 0 0" />
-	</joint>
-	<joint name="kinect2_to_left_kinect_base" type="fixed">
-	  <parent link="middle_kinect_base" />
-	  <child link="left_kinect_base" />
-	  <origin rpy="${PI/2} ${-0.8*PI/2} 0" xyz="0 0 0" />
-	</joint>
 	<joint name="yumi_to_middle_kinect_base" type="fixed">
 	  <parent link="yumi_base_link" />
 	  <child link="middle_kinect_base" />
-	  <origin rpy="0 ${-PI/2} 0" xyz="-0.03 0 0.56" />
+	  <origin rpy="0 ${-0.8*PI/2} 0" xyz="-0.03 0 0.56" />
 	</joint>
 	<joint name="middle_kinect_base_to_kinect2" type="fixed">

Commit message: Updating URDF with optoforce sensors calibration

File: yumi_description/urdf/yumi.urdf (robot description, URDF)
Before this commit: robot yumi, 24 links, 23 joints
Joints:
- joint optodaq_l_sensor_link_joint: origin xyz=0 0 0.033 rpy=0 0 3.14159265359 -> xyz=0 0 -0.033 rpy=3.14159265359 0.0 0.785398163397
- joint optodaq_r_sensor_link_joint: origin xyz=0 0 0.033 rpy=0 0 3.14159265359 -> xyz=0 0 -0.033 rpy=3.14159265359 0.0 0.785398163397
- joint yumi_link_7_l_joint: origin xyz=0 0 0.033 rpy=0 0 3.14159265359 -> xyz=0 0 0.033 rpy=0 3.14159265359 -0.785398163397
- joint yumi_link_7_r_joint: origin xyz=0 0 0.033 rpy=0 0 3.14159265359 -> xyz=0 0 0.033 rpy=0 3.14159265359 -0.785398163397

Commit message: Fixed the yumi joint limits. Added the kinect model properly to the overall model

File: yumi_description/urdf/yumi.urdf (robot description, URDF)
Before this commit: robot yumi, 28 links, 27 joints
Joints:
- joint middle_kinect_base_to_kinect2: origin xyz=0.2 0 0 rpy=-1.57079632679 0 -1.57079632679 -> xyz=0.25 0 -0.1 rpy=-3.14159 0 -1.57079632679
- joint pedestal_to_table: origin xyz=-0.05 0.235 0.05 rpy=0 0 0 -> xyz=0.005 0.235 0.04 rpy=0 0 0
- joint pedestal_to_yumi: origin xyz=-0.0625 0 0.05 rpy=0 0 0 -> xyz=0.0 0 0.05 rpy=0 0 0
- joint yumi_joint_1_l: limit lower=-2.94087978961 upper=2.94087978961 effort=300 velocity=3.14159265359 -> lower=-2.74087978961 upper=2.74087978961 effort=300 velocity=3.14159265359
- joint yumi_joint_1_r: limit lower=-2.94087978961 upper=2.94087978961 effort=300 velocity=3.14159265359 -> lower=-2.74087978961 upper=2.74087978961 effort=300 velocity=3.14159265359
- joint yumi_joint_2_l: limit lower=-2.50454747661 upper=0.759218224618 effort=300 velocity=3.14159265359 -> lower=-2.28454747661 upper=0.539218224618 effort=300 velocity=3.14159265359
- joint yumi_joint_2_r: limit lower=-2.50454747661 upper=0.759218224618 effort=300 velocity=3.14159265359 -> lower=-2.28454747661 upper=0.539218224618 effort=300 velocity=3.14159265359
- joint yumi_joint_3_l: limit lower=-2.15548162621 upper=1.3962634016 effort=300 velocity=3.14159265359 -> lower=-1.95548162621 upper=1.1962634016 effort=300 velocity=3.14159265359
- joint yumi_joint_3_r: limit lower=-2.15548162621 upper=1.3962634016 effort=300 velocity=3.14159265359 -> lower=-1.95548162621 upper=1.1962634016 effort=300 velocity=3.14159265359
- joint yumi_joint_4_l: limit lower=-5.06145483078 upper=5.06145483078 effort=300 velocity=6.98131700798 -> lower=-4.86145483078 upper=4.86145483078 effort=300 velocity=6.98131700798
- joint yumi_joint_4_r: limit lower=-5.06145483078 upper=5.06145483078 effort=300 velocity=6.98131700798 -> lower=-4.86145483078 upper=4.86145483078 effort=300 velocity=6.98131700798
- joint yumi_joint_5_l: limit lower=-1.53588974176 upper=2.40855436775 effort=300 velocity=6.98131700798 -> lower=-1.32588974176 upper=2.19855436775 effort=300 velocity=6.98131700798
- joint yumi_joint_5_r: limit lower=-1.53588974176 upper=2.40855436775 effort=300 velocity=6.98131700798 -> lower=-1.32588974176 upper=2.19855436775 effort=300 velocity=6.98131700798
- joint yumi_joint_6_l: limit lower=-3.99680398707 upper=3.99680398707 effort=300 velocity=6.98131700798 -> lower=-3.89680398707 upper=3.89680398707 effort=300 velocity=6.98131700798
- joint yumi_joint_6_r: limit lower=-3.99680398707 upper=3.99680398707 effort=300 velocity=6.98131700798 -> lower=-3.89680398707 upper=3.89680398707 effort=300 velocity=6.98131700798
- joint yumi_joint_7_l: limit lower=-2.94087978961 upper=2.94087978961 effort=300 velocity=3.14159265359 -> lower=-2.73087978961 upper=2.73087978961 effort=300 velocity=3.14159265359
- joint yumi_joint_7_r: limit lower=-2.94087978961 upper=2.94087978961 effort=300 velocity=3.14159265359 -> lower=-2.73087978961 upper=2.73087978961 effort=300 velocity=3.14159265359
- joint yumi_to_middle_kinect_base: origin xyz=-0.03 0 0.56 rpy=0 -1.25663706144 0 -> xyz=-0.03 0 0.7 rpy=0 -1.09955742876 0

File: yumi_description/urdf/yumi.urdf.xacro (robot description, xacro)
@@ -53,5 +53,5 @@
 	  <parent link="yumi_pedestal" />
 	  <child link="table" />
-	  <origin rpy="0 0 0" xyz="-0.05 0.235 ${yumi_height + 0.01}" />
+	  <origin rpy="0 0 0" xyz="0.005 0.235 ${yumi_height }" />
 	</joint>
 	<link name="table">
@@ -116,9 +116,9 @@
 	  <parent link="yumi_pedestal" />
 	  <child link="yumi_base_link" />
-	  <origin rpy="0 0 0" xyz="-0.0625 0 ${yumi_height+0.01}" />
+	  <origin rpy="0 0 0" xyz="0.0 0 ${yumi_height}" />
 	</joint>
-	<link name="kinect2">
+	<link name="kinect2_link">
 	  <visual>
-	    <origin xyz="0 0 0" rpy="0 0 0" />
+	    <origin xyz="0 0 0" rpy="${PI/2} 0 0" />
 	    <geometry>
 	      <mesh scale="0.001 0.001 0.001" filename="package://yumi_description/meshes/accesories/KinectXboxOne.stl"/>
@@ -138,5 +138,5 @@
 	      <origin xyz="0 0 0" rpy="0 0 0" />
 	      <geometry>
-	        <box size="0.4 0.15 0.02" />
+	        <box size="0.6 0.15 0.02" />
 	      </geometry>
 	      <material name="Grey" />
@@ -147,5 +147,5 @@
 	        <box size="0.4 0.15 0.02" />
 	      </geometry>
-	      <material name="Grey" />
+	      <material name="Grey" /> ${-PI}
 	    </collision> -->
 	</link>
@@ -153,10 +153,22 @@
 	  <parent link="yumi_base_link" />
 	  <child link="middle_kinect_base" />
-	  <origin rpy="0 ${-0.8*PI/2} 0" xyz="-0.03 0 0.56" />
+	  <origin rpy="0 ${-0.7*PI/2} 0" xyz="0.00 0 0.73" />
+	</joint>
+         <link name="kinect2_rotation">
+          </link>
+        <!--<joint name="kinect2_to_kinect2_link" type="fixed">
+	  <parent link="kinect2" />
+	  <child link="kinect2_link" />
+	  <origin rpy="0 0 0" xyz="0.00 0 0.0" />  -3.77  0 ${kinect_zrotation_fix}
+	</joint> -->
+        <joint name="kinect2_link_to_kinect2_rotation" type="fixed">
+	  <parent link="kinect2_rotation" />
+	  <child link="kinect2_link" />
+	  <origin rpy="0.0 0.0 ${-PI/2}" xyz="0.0 0.0 0.0" />
 	</joint>
 	<joint name="middle_kinect_base_to_kinect2" type="fixed">
-	  <parent link="middle_kinect_base" />
-	  <child link="kinect2" />
-	  <origin rpy="${-PI/2} 0 ${kinect_zrotation_fix}" xyz="0.2 0 0" />
+	  <parent link="yumi_base_link" />
+	  <child link="kinect2_rotation" />
+	  <origin rpy="0.0 2.4426 0.0" xyz="0.14 -0.06 0.92" />
 	</joint>
 </robot>

File: yumi_description/urdf/yumi.xacro (robot description, xacro)
@@ -43,5 +43,5 @@
       <origin xyz="0.05355 -0.0725 0.41492" rpy="-0.9795   -0.5682   -2.3155"/>
       <axis xyz="0 0 1"/>
-      <limit lower="${-168.5 * PI / 180}" upper="${168.5 * PI / 180}"
+      <limit lower="${-158.5 * PI / 180}" upper="${158.5 * PI / 180}"
              effort="${max_effort}" velocity="${180 * PI / 180}" />
       <dynamics damping="${joint_damping}"/>
@@ -74,5 +74,5 @@
       <origin xyz="0.03 0.0 0.1" rpy="${PI / 2} 0.0 0.0"/>
       <axis xyz="0 0 1"/>
-      <limit lower="${-143.5 * PI / 180}" upper="${43.5 * PI / 180}"
+      <limit lower="${-133.5 * PI / 180}" upper="${33.5 * PI / 180}"
              effort="${max_effort}" velocity="${180 * PI / 180}" />
       <dynamics damping="${joint_damping}"/>
@@ -105,5 +105,5 @@
         <origin xyz="-0.03 0.17283 0.0" rpy="${-PI / 2} 0.0 0.0"/>
         <axis xyz="0 0 1"/>
-        <limit lower="${-168.5 * PI / 180}" upper="${168.5 * PI / 180}"
+        <limit lower="${-158.5 * PI / 180}" upper="${158.5 * PI / 180}"
                effort="${max_effort}" velocity="${180 * PI / 180}" />
         <dynamics damping="${joint_damping}"/>
@@ -136,5 +136,5 @@
       <origin xyz="-0.04188 0.0 0.07873" rpy="${PI / 2} ${- PI / 2} 0.0"/>
       <axis xyz="0 0 1"/>
-      <limit lower="${-123.5 * PI / 180}" upper="${80 * PI / 180}"
+      <limit lower="${-113.5 * PI / 180}" upper="${70 * PI / 180}"
              effort="${max_effort}" velocity="${180 * PI / 180}" />
       <dynamics damping="${joint_damping}"/>
@@ -167,5 +167,5 @@
       <origin xyz="0.0405 0.16461 0.0" rpy="-${PI / 2} 0.0 0.0"/>
       <axis xyz="0 0 1"/>
-      <limit lower="${-290 * PI / 180}" upper="${290 * PI / 180}"
+      <limit lower="${-280 * PI / 180}" upper="${280 * PI / 180}"
              effort="${max_effort}" velocity="${400 * PI / 180}" />
       <dynamics damping="${joint_damping}"/>
@@ -198,5 +198,5 @@
       <origin xyz="-0.027 0 0.10039" rpy="${PI / 2} 0.0 0.0"/>
       <axis xyz="0 0 1"/>
-      <limit lower="${-88 * PI / 180}" upper="${138 * PI / 180}"
+      <limit lower="${-78 * PI / 180}" upper="${128 * PI / 180}"
              effort="${max_effort}" velocity="${400 * PI / 180}" />
       <dynamics damping="${joint_damping}"/>
@@ -229,5 +229,5 @@
       <origin xyz="0.027 0.029 0.0" rpy="-${PI / 2} 0.0 0.0"/>
       <axis xyz="0 0 1"/>
-      <limit lower="${-229 * PI / 180}" upper="${229 * PI / 180}"
+      <limit lower="${-219 * PI / 180}" upper="${219 * PI / 180}"
              effort="${max_effort}" velocity="${400 * PI / 180}" />
       <dynamics damping="${joint_damping}"/>
@@ -261,5 +261,5 @@
       <origin xyz="0.05355 0.07250 0.41492" rpy="0.9781 -0.5716 2.3180"/>
       <axis xyz="0 0 1"/>
-      <limit lower="${-168.5 * PI / 180}" upper="${168.5 * PI / 180}"
+      <limit lower="${-158.5 * PI / 180}" upper="${158.5 * PI / 180}"
              effort="${max_effort}" velocity="${180 * PI / 180}" />
       <dynamics damping="${joint_damping}"/>
@@ -292,5 +292,5 @@
       <origin xyz="0.03 0.0 0.1" rpy="${PI / 2} 0.0 0.0"/>
       <axis xyz="0 0 1"/>
-      <limit lower="${-143.5 * PI / 180}" upper="${43.5 * PI / 180}"
+      <limit lower="${-133.5 * PI / 180}" upper="${33.5 * PI / 180}"
              effort="${max_effort}" velocity="${180 * PI / 180}" />
       <dynamics damping="${joint_damping}"/>
@@ -323,5 +323,5 @@
       <origin xyz="-0.03 0.17283 0.0" rpy="-${PI / 2} 0.0 0.0"/>
       <axis xyz="0 0 1"/>
-      <limit lower="${-168.5 * PI / 180}" upper="${168.5 * PI / 180}"
+      <limit lower="${-158.5 * PI / 180}" upper="${158.5 * PI / 180}"
              effort="${max_effort}" velocity="${180 * PI / 180}" />
       <dynamics damping="${joint_damping}"/>
@@ -354,5 +354,5 @@
       <origin xyz="-0.04188 0.0 0.07873" rpy="${PI / 2} -${PI / 2} 0.0"/>
       <axis xyz="0 0 1"/>
-      <limit lower="${-123.5 * PI / 180}" upper="${80 * PI / 180}"
+      <limit lower="${-115.5 * PI / 180}" upper="${70 * PI / 180}"
              effort="${max_effort}" velocity="${180 * PI / 180}" />
       <dynamics damping="${joint_damping}"/>
@@ -385,5 +385,5 @@
       <origin xyz="0.0405 0.16461 0.0" rpy="-${PI / 2} 0.0 0.0"/>
       <axis xyz="0 0 1"/>
-      <limit lower="${-290 * PI / 180}" upper="${290 * PI / 180}"
+      <limit lower="${-280 * PI / 180}" upper="${280 * PI / 180}"
              effort="${max_effort}" velocity="${400 * PI / 180}" />
       <dynamics damping="${joint_damping}"/>
@@ -416,5 +416,5 @@
       <origin xyz="-0.027 0 0.10039" rpy="${PI / 2} 0.0 0.0"/>
       <axis xyz="0 0 1"/>
-      <limit lower="${-88 * PI / 180}" upper="${138 * PI / 180}"
+      <limit lower="${-80 * PI / 180}" upper="${128 * PI / 180}"
              effort="${max_effort}" velocity="${400 * PI / 180}" />
       <dynamics damping="${joint_damping}"/>
@@ -447,5 +447,5 @@
       <origin xyz="0.027 0.029 0.0" rpy="${-PI / 2} 0.0 0.0"/>
       <axis xyz="0 0 1"/>
-      <limit lower="${-229 * PI / 180}" upper="${229 * PI / 180}"
+      <limit lower="${-219 * PI / 180}" upper="${219 * PI / 180}"
              effort="${max_effort}" velocity="${400 * PI / 180}" />
       <dynamics damping="${joint_damping}"/>

Commit message: Fixes for world vs robot_centric moveit planning frame issue

File: yumi_description/urdf/yumi.urdf (robot description, URDF)
Before this commit: robot yumi, 28 links, 27 joints
Links:
- removed link kinect2
- added link kinect2_link; visual mesh filename=package://yumi_description/meshes/accesories/KinectXboxOne.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 scale=0.001 0.001 0.001
- added link kinect2_rotation
- link middle_kinect_base: geometry visual box size=0.6 0.15 0.02
Joints:
- added joint kinect2_link_to_kinect2_rotation: type fixed, parent kinect2_rotation, child kinect2_link, origin xyz=0.0 0.0 0.0 rpy=0.0 0.0 -1.57079632679
- joint middle_kinect_base_to_kinect2: child kinect2 -> kinect2_rotation; origin xyz=0.25 0 -0.1 rpy=-3.14159 0 -1.57079632679 -> xyz=0.14 -0.06 0.92 rpy=0.0 2.4426 0.0; parent middle_kinect_base -> yumi_base_link
- joint yumi_joint_1_l: limit lower=-2.74087978961 upper=2.74087978961 effort=300 velocity=3.14159265359 -> lower=-2.76634686441 upper=2.76634686441 effort=300 velocity=3.14159265359
- joint yumi_joint_1_r: limit lower=-2.74087978961 upper=2.74087978961 effort=300 velocity=3.14159265359 -> lower=-2.76634686441 upper=2.76634686441 effort=300 velocity=3.14159265359
- joint yumi_joint_2_l: limit lower=-2.28454747661 upper=0.539218224618 effort=300 velocity=3.14159265359 -> lower=-2.33001455141 upper=0.584685299418 effort=300 velocity=3.14159265359
- joint yumi_joint_2_r: limit lower=-2.28454747661 upper=0.539218224618 effort=300 velocity=3.14159265359 -> lower=-2.33001455141 upper=0.584685299418 effort=300 velocity=3.14159265359
- joint yumi_joint_3_l: limit lower=-1.95548162621 upper=1.1962634016 effort=300 velocity=3.14159265359 -> lower=-2.01585528605 upper=1.2217304764 effort=300 velocity=3.14159265359
- joint yumi_joint_3_r: limit lower=-1.95548162621 upper=1.1962634016 effort=300 velocity=3.14159265359 -> lower=-1.98094870101 upper=1.2217304764 effort=300 velocity=3.14159265359
- joint yumi_joint_4_l: limit lower=-4.86145483078 upper=4.86145483078 effort=300 velocity=6.98131700798 -> lower=-4.88692190558 upper=4.88692190558 effort=300 velocity=6.98131700798
- joint yumi_joint_4_r: limit lower=-4.86145483078 upper=4.86145483078 effort=300 velocity=6.98131700798 -> lower=-4.88692190558 upper=4.88692190558 effort=300 velocity=6.98131700798
- joint yumi_joint_5_l: limit lower=-1.32588974176 upper=2.19855436775 effort=300 velocity=6.98131700798 -> lower=-1.3962634016 upper=2.23402144255 effort=300 velocity=6.98131700798
- joint yumi_joint_5_r: limit lower=-1.32588974176 upper=2.19855436775 effort=300 velocity=6.98131700798 -> lower=-1.36135681656 upper=2.23402144255 effort=300 velocity=6.98131700798
- joint yumi_joint_6_l: limit lower=-3.89680398707 upper=3.89680398707 effort=300 velocity=6.98131700798 -> lower=-3.82227106187 upper=3.82227106187 effort=300 velocity=6.98131700798
- joint yumi_joint_6_r: limit lower=-3.89680398707 upper=3.89680398707 effort=300 velocity=6.98131700798 -> lower=-3.82227106187 upper=3.82227106187 effort=300 velocity=6.98131700798
- joint yumi_joint_7_l: limit lower=-2.73087978961 upper=2.73087978961 effort=300 velocity=3.14159265359 -> lower=-2.76634686441 upper=2.76634686441 effort=300 velocity=3.14159265359
- joint yumi_joint_7_r: limit lower=-2.73087978961 upper=2.73087978961 effort=300 velocity=3.14159265359 -> lower=-2.76634686441 upper=2.76634686441 effort=300 velocity=3.14159265359
- joint yumi_to_middle_kinect_base: origin xyz=-0.03 0 0.7 rpy=0 -1.09955742876 0 -> xyz=0.00 0 0.73 rpy=0 -1.09955742876 0

File: yumi_description/urdf/yumi.urdf.xacro (robot description, xacro)
@@ -23,9 +23,10 @@
 		<origin xyz="0 0 0.007" rpy="0 0 ${PI}" />
 	</xacro:yumi_servo_gripper>
+        <!--
 	<xacro:property name="yumi_setup" value="$(arg yumi_setup)" />
 	<xacro:if value="${yumi_setup == 'robot_centric'}">
-		<!-- Pure YuMi URDF, with no joints connecting it to any other robot or pedestal. Neither accessories. -->
-	</xacro:if>
-	<xacro:if value="${yumi_setup == 'default'}">
+		 Pure YuMi URDF, with no joints connecting it to any other robot or pedestal. Neither accessories.
+	</xacro:if> -->
+	<!--<xacro:if value="${yumi_setup == 'default'}">
 		<link name="world"/>
 		<joint name="world_to_pedestal" type="fixed">
@@ -34,5 +35,5 @@
 			<origin rpy="0 0 0" xyz="0 0 ${pedestal_height}" />
 		</joint>
-	</xacro:if>
+	</xacro:if> -->
 	<xacro:property name="pedestal_height" value="0.92" />
 	<xacro:property name="pedestal_xrotation_fix" value="${- PI / 2.0}" />
