Commit message: Disable logging by default. Set parameter for exponential smoothing. Define folding objects in urdf for motion planner

File: yumi_description/urdf/yumi.urdf (robot description, URDF)
Before this commit: robot yumi, 24 links, 23 joints
Links:
- added link fold_case_sensor_link; visual cylinder length=0.24 radius=0.06
- added link rod_piece_sensor_link; visual cylinder length=0.16 radius=0.06
Joints:
- removed joint yumi_link_7_l_joint
- removed joint yumi_link_7_r_joint
- added joint yumi_link_7_l_joint_daq: type fixed, parent yumi_link_7_l, child optodaq_l_sensor_link, origin xyz=0 0 0.033 rpy=0 3.14159265359 -0.785398163397
- added joint yumi_link_7_r_joint_daq: type fixed, parent yumi_link_7_r, child optodaq_r_sensor_link, origin xyz=0 0 0.033 rpy=0 3.14159265359 -0.785398163397
- joint gripper_l_joint: axis -1 0 0 -> (none); child gripper_l_finger_r -> rod_piece_sensor_link; limit lower=0 upper=0.025 effort=20 velocity=2 -> (none); origin xyz=0 -0.0065 0.0837 rpy=0 0 0 -> xyz=0 0 0 rpy=0 0 0; parent gripper_l_base -> gripper_l; type prismatic -> fixed
- joint gripper_r_joint: axis -1 0 0 -> (none); child gripper_r_finger_r -> fold_case_sensor_link; limit lower=0 upper=0.025 effort=20 velocity=2 -> (none); origin xyz=0 -0.0065 0.0837 rpy=0 0 0 -> xyz=0 0 0 rpy=0 0 0; parent gripper_r_base -> gripper_r; type prismatic -> fixed

File: yumi_description/urdf/yumi.urdf.xacro (robot description, xacro)
@@ -11,4 +11,7 @@
   <!--Import the yumi optodaq sensors macro -->
   <xacro:include filename="$(find yumi_description)/urdf/Extras/yumi_optodaq_sensors.xacro"/>
+  <!--Import folding macros -->
+  <xacro:include filename="$(find yumi_description)/urdf/Extras/yumi_fold_case.xacro"/>
+  <xacro:include filename="$(find yumi_description)/urdf/Extras/yumi_rod.xacro"/>
   <!-- Import Gazebo plugins -->
   <xacro:include filename="$(find yumi_description)/urdf/Gazebo/gazebo.urdf.xacro"/>
@@ -31,4 +34,12 @@
    <origin xyz="0 0 -0.033" rpy="${PI} 0.0 ${PI/4}" />
  </xacro:yumi_servo_gripper>
+ <!-- Surface piece -->
+ <xacro:yumi_fold_case name="fold_case" parent="gripper_r">
+   <origin xyz="0 0 0" rpy="0 0 0" />
+ </xacro:yumi_fold_case>
+ <!-- Rod piece -->
+ <xacro:yumi_rod name="rod_piece" parent="gripper_l">
+   <origin xyz="0 0 0" rpy="0 0 0" />
+ </xacro:yumi_rod>
   <xacro:property name="yumi_setup" value="$(arg yumi_setup)" />
   <xacro:if value="${yumi_setup == 'robot_centric'}">

Commit message: fixed frame name has been changed. Some parameter changes in moveit in order to prevent motion abort during execution

File: yumi_description/urdf/yumi.urdf (robot description, URDF)
Before this commit: robot yumi, 30 links, 29 joints
Links:
- link middle_kinect_base: geometry visual box size=0.6 0.27 0.02

File: yumi_description/urdf/yumi.urdf.xacro (robot description, xacro)
@@ -156,5 +156,5 @@
 	      <origin xyz="0 0 0" rpy="0 0 0" />
 	      <geometry>
-	        <box size="0.6 0.15 0.02" />
+	        <box size="0.6 0.27 0.02" />
 	      </geometry>
 	      <material name="Grey" />

Commit message: attach yumi_base_lnk to world to solve the couldn't find chain problem for trac-ik

File: yumi_description/urdf/yumi.urdf (robot description, URDF)
Before this commit: robot yumi, 22 links, 21 joints
Links:
- added link world
Joints:
- added joint world_to_base_link: type fixed, parent world, child yumi_base_link

Commit message: fixed the offset from world to base_link

File: yumi_description/urdf/yumi.urdf (robot description, URDF)
Before this commit: robot yumi, 23 links, 22 joints
Joints:
- joint world_to_base_link: origin (none) -> xyz=0 0 0.1 rpy=0 0 0
