Commit message: Fix to the yumi grippers dettachment problem in Gazebo

File: yumi_description/urdf/Grippers/yumi_servo_gripper.xacro (robot description, xacro)
@@ -5,4 +5,5 @@
     <!-- Import Transmissions -->
     <xacro:include filename="$(find yumi_description)/urdf/Grippers/yumi_servo_gripper.transmission.xacro" />
+    <xacro:include filename="$(find hector_xacro_tools)/urdf/inertia_tensors.urdf.xacro" />
     <!-- some constants -->
     <xacro:property name="joint_damping" value="0.5" />
@@ -49,9 +50,5 @@
     </joint>
     <link name="${name}_finger_r">
-      <inertial>
-        <origin xyz="0 0 0" rpy="0 0 0"/>
-        <mass value="0.01"/>
-        <inertia ixx="0.000001"  ixy="0"  ixz="0" iyy="0.000001" iyz="0" izz="0.000001" />
-      </inertial>
+      <xacro:inertial_cuboid mass="0.1" x_length="0.05" y_length="0.05" z_length="0.05" />
       <visual>
         <origin xyz="0 0 0" rpy="0 0 0"/>
@@ -81,9 +78,5 @@
     </joint>
     <link name="${name}_finger_l">
-      <inertial>
-        <origin xyz="0 0 0" rpy="0 0 0"/>
-        <mass value="0.01"/>
-        <inertia ixx="0.000001"  ixy="0"  ixz="0" iyy="0.000001" iyz="0" izz="0.000001" />
-      </inertial>
+      <xacro:inertial_cuboid mass="0.1" x_length="0.05" y_length="0.05" z_length="0.05" />
       <visual>
         <origin xyz="0 0 0" rpy="0 0 0"/>

Commit message: Changes to the yumi model that compansate various errors. Added a coarse finger model for easier approach to objects (Credits: Rika Antonova)

File: yumi_description/urdf/Grippers/yumi_servo_gripper.xacro (robot description, xacro)
@@ -11,4 +11,13 @@
     <xacro:property name="max_gripper_effort" value="20"/>
     <xacro:property name="max_gripper_velocity" value="2"/>
+    <!-- xacro:property name="finger_scale" value="1.0" / -->
+    <xacro:property name="finger_offset_y" value="0" />
+    <xacro:property name="finger_offset_z" value="-0.005" />
+    <!-- brown fingers were large in the CAD model, so scale down-->
+    <xacro:property name="finger_scale" value="0.001" />
+    <!-- For yumi_finger_for_optoforce.stl -->
+    <!-- xacro:property name="finger_scale" value="0.001" / -->
+    <!-- xacro:property name="finger_offset_y" value="0.008" / -->
+    <!-- xacro:property name="finger_offset_z" value="-0.005" / -->
   <xacro:macro name="yumi_servo_gripper" params="parent name hardware_interface *origin">
     <!--joint between {parent} and base-->
@@ -52,14 +61,14 @@
       <xacro:inertial_cuboid mass="0.1" x_length="0.05" y_length="0.05" z_length="0.05" />
       <visual>
-        <origin xyz="0 0 0" rpy="0 0 0"/>
+        <origin xyz="0 ${finger_offset_y} ${finger_offset_z}" rpy="0 0 0"/>
         <geometry>
-          <mesh filename="package://yumi_description/meshes/gripper/finger.stl"/>
+          <mesh scale="${finger_scale} ${finger_scale} ${finger_scale}" filename="package://yumi_description/meshes/gripper/coarse/brown_finger.stl"/>
         </geometry>
         <material name="Blue"/>
       </visual>
       <collision>
-        <origin xyz="0 0 0" rpy="0 0 0"/>
+        <origin xyz="0 ${finger_offset_y} ${finger_offset_z}" rpy="0 0 0"/>
         <geometry>
-          <mesh filename="package://yumi_description/meshes/gripper/coarse/finger.stl"/>
+          <mesh scale="${finger_scale} ${finger_scale} ${finger_scale}" filename="package://yumi_description/meshes/gripper/coarse/brown_finger.stl"/>
         </geometry>
         <material name="Blue"/>
@@ -80,14 +89,14 @@
       <xacro:inertial_cuboid mass="0.1" x_length="0.05" y_length="0.05" z_length="0.05" />
       <visual>
-        <origin xyz="0 0 0" rpy="0 0 0"/>
+        <origin xyz="0 ${finger_offset_y} ${finger_offset_z}" rpy="0 0 0"/>
         <geometry>
-          <mesh filename="package://yumi_description/meshes/gripper/finger.stl"/>
+          <mesh scale="${finger_scale} ${finger_scale} ${finger_scale}" filename="package://yumi_description/meshes/gripper/coarse/brown_finger.stl"/>
         </geometry>
         <material name="Blue"/>
       </visual>
       <collision>
-        <origin xyz="0 0 0" rpy="0 0 0"/>
+        <origin xyz="0 ${finger_offset_y} ${finger_offset_z}" rpy="0 0 0"/>
         <geometry>
-          <mesh filename="package://yumi_description/meshes/gripper/coarse/finger.stl"/>
+          <mesh scale="${finger_scale} ${finger_scale} ${finger_scale}" filename="package://yumi_description/meshes/gripper/coarse/brown_finger.stl"/>
         </geometry>
         <material name="Blue"/>

File: yumi_description/urdf/yumi.urdf (robot description, URDF)
Before this commit: robot yumi, 29 links, 28 joints
Links:
- added link world
- link gripper_l_finger_l: mass 0.01 -> 0.1; geometry collision mesh filename=package://yumi_description/meshes/gripper/coarse/brown_fing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 scale=0.001 0.001 0.001; visual mesh filename=package://yumi_description/meshes/gripper/coarse/brown_fing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 scale=0.001 0.001 0.001
- link gripper_l_finger_r: mass 0.01 -> 0.1; geometry collision mesh filename=package://yumi_description/meshes/gripper/coarse/brown_fing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 scale=0.001 0.001 0.001; visual mesh filename=package://yumi_description/meshes/gripper/coarse/brown_fing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 scale=0.001 0.001 0.001
- link gripper_r_finger_l: mass 0.01 -> 0.1; geometry collision mesh filename=package://yumi_description/meshes/gripper/coarse/brown_fing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 scale=0.001 0.001 0.001; visual mesh filename=package://yumi_description/meshes/gripper/coarse/brown_fing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 scale=0.001 0.001 0.001
- link gripper_r_finger_r: mass 0.01 -> 0.1; geometry collision mesh filename=package://yumi_description/meshes/gripper/coarse/brown_fing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 scale=0.001 0.001 0.001; visual mesh filename=package://yumi_description/meshes/gripper/coarse/brown_fing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 scale=0.001 0.001 0.001
Joints:
- added joint world_to_pedestal: type fixed, parent world, child yumi_pedestal, origin xyz=0 0 0.92 rpy=0 0 0
- joint middle_kinect_base_to_kinect2: origin xyz=0.14 -0.06 0.92 rpy=0.0 2.4426 0.0 -> xyz=0.27 0 0.81 rpy=0.0 2.4426 0.0
- joint pedestal_to_yumi: origin xyz=0.0 0 0.05 rpy=0 0 0 -> xyz=0.0 0 0.04 rpy=0 0 0
- joint yumi_base_link_to_body: origin xyz=0 0 0 rpy=0 0 0 -> xyz=0 0 0 rpy=0 -0.0175 0
- joint yumi_to_middle_kinect_base: origin xyz=0.00 0 0.73 rpy=0 -1.09955742876 0 -> xyz=0.10 0 0.71 rpy=0 -0.911061869541 0

File: yumi_description/urdf/yumi.urdf.xacro (robot description, xacro)
@@ -28,5 +28,4 @@
 		 Pure YuMi URDF, with no joints connecting it to any other robot or pedestal. Neither accessories.
 	</xacro:if> -->
-	<!--<xacro:if value="${yumi_setup == 'default'}">
 		<link name="world"/>
 		<joint name="world_to_pedestal" type="fixed">
@@ -35,5 +34,4 @@
 			<origin rpy="0 0 0" xyz="0 0 ${pedestal_height}" />
 		</joint>
-	</xacro:if> -->
 	<xacro:property name="pedestal_height" value="0.92" />
 	<xacro:property name="pedestal_xrotation_fix" value="${- PI / 2.0}" />
@@ -42,4 +40,5 @@
 	<xacro:property name="yumi_parent" value="yumi_pedestal" />
 	<xacro:property name="kinect_zrotation_fix" value="${- PI / 2.0}" />
+	<xacro:property name="table_top_offset" value="0.005" />
 	<link name="yumi_pedestal">
 	  <visual>
@@ -96,5 +95,6 @@
 	  <parent link="table_extension_bottom" />
 	  <child link="table_extension_top" />
-	  <origin rpy="0 0 0" xyz="0 0 0.005" />
+	  <!-- origin rpy="0 0 0" xyz="0 0 0.005" / -->
+	  <origin rpy="0 0 0" xyz="0 0 ${table_top_offset}" />
 	</joint>
 	<link name="table_extension_top">
@@ -123,4 +123,5 @@
 	    <origin xyz="0 0 0" rpy="${PI/2} 0 0" />
 	    <geometry>
+	     <!-- mesh scale="0.001 0.001 0.001" filename="package://yumi_description/meshes/accesories/KinectXboxOne.stl"/ -->
 	      <mesh scale="0.001 0.001 0.001" filename="package://yumi_description/meshes/accesories/KinectXboxOne.stl"/>
 	    </geometry>
@@ -135,4 +136,20 @@
 	  </collision> -->
 	</link>
+	<!-- <link name="kinectp_link">
+	  <visual>
+	    <origin xyz="0 0 0" rpy="${PI/2} 0 0" />
+	    <geometry>
+	     <mesh scale="0.001 0.001 0.001" filename="package://yumi_description/meshes/accesories/KinectXboxOne.stl"/>
+	    </geometry>
+	    <material name="Black" />
+	  </visual>
+	  <collision>
+	    <origin xyz="0 0 0" rpy="0 0 0" />
+	    <geometry>
+	      <mesh scale="0.001 0.001 0.001" filename="package://yumi_description/meshes/accesories/KinectXboxOne.stl"/>
+	    </geometry>
+	    <material name="Black" />
+	  </collision>
+	</link> -->
 	<link name="middle_kinect_base">
 	    <visual>
@@ -154,14 +171,15 @@
 	  <parent link="yumi_base_link" />
 	  <child link="middle_kinect_base" />
-	  <origin rpy="0 ${-0.7*PI/2} 0" xyz="0.00 0 0.73" />
+	  <origin rpy="0 ${-0.58*PI/2} 0" xyz="0.10 0 0.71" />
+	  <!-- origin rpy="0 ${-0.7*PI/2} 0" xyz="0.00 0 0.73" / -->
 	</joint>
-         <link name="kinect2_rotation">
-          </link>
-        <!--<joint name="kinect2_to_kinect2_link" type="fixed">
+    <link name="kinect2_rotation">
+    </link>
+    <!--<joint name="kinect2_to_kinect2_link" type="fixed">
 	  <parent link="kinect2" />
 	  <child link="kinect2_link" />
 	  <origin rpy="0 0 0" xyz="0.00 0 0.0" />  -3.77  0 ${kinect_zrotation_fix}
 	</joint> -->
-        <joint name="kinect2_link_to_kinect2_rotation" type="fixed">
+    <joint name="kinect2_link_to_kinect2_rotation" type="fixed">
 	  <parent link="kinect2_rotation" />
 	  <child link="kinect2_link" />
@@ -171,5 +189,11 @@
 	  <parent link="yumi_base_link" />
 	  <child link="kinect2_rotation" />
-	  <origin rpy="0.0 2.4426 0.0" xyz="0.14 -0.06 0.92" />
+	  <!-- origin rpy="0.0 2.4426 0.0" xyz="0.14 -0.06 0.92" / -->
+	  <origin rpy="0.0 2.4426 0.0" xyz="0.27 0 0.81" />
 	</joint>
+<!--	<joint name="yumi_base_link_to_kinectp_link" type="fixed">
+	  <parent link="yumi_base_link" />
+	  <child link="kinectp_link" />
+	  <origin rpy="-2.99236 0.04977 -1.55351" xyz="0.227 0.014 0.7065" />
+	</joint> -->
 </robot>

File: yumi_description/urdf/yumi.xacro (robot description, xacro)
@@ -8,4 +8,6 @@
   <xacro:property name="joint_damping" value="0.5" />
   <xacro:property name="max_effort" value="300"/>
+  <!-- Yumi body has tiled back by ~1-2deg (-0.0175 to -0.035 rad) -->
+  <xacro:property name="yumi_body_tilt" value="-0.0175"/>
   <xacro:macro name="yumi" params="parent name hardware_interface *origin">
     <link name="yumi_base_link"></link>
@@ -13,5 +15,5 @@
       <parent link="yumi_base_link"/>
       <child link="${name}_body"/>
-      <origin xyz="0 0 0" rpy="0 0 0"/>
+      <origin xyz="0 0 0" rpy="0 ${yumi_body_tilt} 0"/>
     </joint>
     <link name="${name}_body">
